File: Schematics/MiniSumoPCB/MiniSumoPCB.kicad_sch (KiCad schematic)
At the start: 50 parts, among them J1 Alimentacion, J18 Servo, J2 AUX_12, J3 MOTOR_A, J4 MOTOR_B, J5 UART, J6 Micro_SD_Card, J8 POWER_OUT_1, Q1 IRLR8726, Q2 IRLM2502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

Commit message: Target tracking
Parts:
- R22: value 680 -> 220
- R23: value 2k2 -> 220
Other:
- note added: "D3:2.2 D1:2.4"
Changed lines of the file:
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@@
     (effects (font (size 3 3) (thickness 0.6) bold) (justify left bottom))
+  )
+  (text "D3:2.2\nD1:2.4" (at 240.03 86.995 0)
+    (effects (font (size 1.27 1.27)) (justify left bottom))
   )
   (text "Todo:\n-----------\n- Leds de estado\n- Salida Servo PWM (x2)\n- Salida High-Power (MOSFET)\n- Control WS2812? (1 Pin)\n- Salida I2c\n"
@@
       (effects (font (size 1.27 1.27)) (justify right))
     )
-    (property "Value" "680" (at 253.238 75.3622 0)
+    (property "Value" "220" (at 253.238 75.3622 0)
       (effects (font (size 1.27 1.27)) (justify right))
     )
@@
   (symbol (lib_id "Device:R") (at 260.35 73.66 0) (mirror y) (unit 1)
     (in_bom yes) (on_board yes) (dnp no) (fields_autoplaced)
-    (property "Reference" "R23" (at 262.128 73.025 0)
-      (effects (font (size 1.27 1.27)) (justify right))
-    )
-    (property "Value" "2k2" (at 262.128 75.565 0)
-      (effects (font (size 1.27 1.27)) (justify right))
-    )
+    (property "Reference" "R23" (at 262.89 72.39 0)
+      (effects (font (size 1.27 1.27)) (justify right))
+    )
+    (property "Value" "220" (at 262.89 74.93 0)
+      (effects (font (size 1.27 1.27)) (justify right))
+    )
